File: Hardware/GaggiaBoard_V3/KiCad/Project/GaggiaBoard_V3.kicad_pcb (KiCad board)
At the start: 2 copper layers, 45 x 100 mm, 80 parts, among them IC1 LD1117AS, J1 Display, J10 PIN262409-1, J11 PIN262409-1, J12 PIN262409-1, J13 PIN262409-1, J14 1x20 Female Header 2.54mm, J15 1x20 Female Header 2.54mm, J2 ToFnLED (Vertical Qwiic), J27 UART1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

Commit message: KiCad project and model updates
Parts:
- J14, J15: footprint Connector_PinSocket_2.54mm:PinSocket_1x20_P2.54mm_Vertical -> GaggiaBoard_V3:1x20_P2.54mm_Female_Vertical
Changed lines of the file:
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@@
     )
   )
-  (footprint "Connector_PinSocket_2.54mm:PinSocket_1x20_P2.54mm_Vertical" (layer "F.Cu")
+  (footprint "GaggiaBoard_V3:1x20_P2.54mm_Female_Vertical" (layer "F.Cu")
     (at 158.623 57.15)
     (descr "Through hole straight socket strip, 1x20, 2.54mm pitch, single row (from Kicad 4.0.7), script generated")
@@
     (property "ki_keywords" "connector")
     (attr through_hole)
-    (fp_text reference "J14" (at -2.286 0) (layer "F.SilkS")
+    (fp_text reference "J14" (at 0 -2.77) (layer "F.SilkS")
         (effects (font (size 1 1) (thickness 0.15)))
     )
@@
     )
   )
-  (footprint "Connector_PinSocket_2.54mm:PinSocket_1x20_P2.54mm_Vertical" (layer "F.Cu")
+  (footprint "GaggiaBoard_V3:1x20_P2.54mm_Female_Vertical" (layer "F.Cu")
     (at 143.383 57.15)
     (descr "Through hole straight socket strip, 1x20, 2.54mm pitch, single row (from Kicad 4.0.7), script generated")
@@
     (property "ki_keywords" "connector")
     (attr through_hole)
-    (fp_text reference "J15" (at -2.413 -0.127) (layer "F.SilkS")
+    (fp_text reference "J15" (at 0 -2.77) (layer "F.SilkS")
         (effects (font (size 1 1) (thickness 0.15)))
     )
@@
       (net 11 "AC_N") (pinfunction "AC_N") (pintype "bidirectional") (solder_mask_margin 0.1016))
     (model "${KIPRJMOD}/GaggiaBoard_V3.pretty/3D/IRM-10-5-2.wrl"
-      (offset (xyz -23.48 -61.67 0))
+      (offset (xyz -0.13 0 -0.09))
       (scale (xyz 0.3937 0.3937 0.3937))
       (rotate (xyz 0 0 0))
@@
         (effects (font (size 0.23368 0.23368) (thickness 0.02032)) (justify left bottom))
     )
-    (fp_text user "direction of pcb" (at 0.4 0.4 180) (layer "Cmts.User")
+    (fp_text user "wavesoldering" (at 0.4 -0.5 180) (layer "Cmts.User")
         (effects (font (size 0.23368 0.23368) (thickness 0.02032)) (justify left bottom))
     )
-    (fp_text user "wavesoldering" (at 0.4 -0.5 180) (layer "Cmts.User")
+    (fp_text user "direction of pcb" (at 0.4 0.4 180) (layer "Cmts.User")
         (effects (font (size 0.23368 0.23368) (thickness 0.02032)) (justify left bottom))
     )
