File: Hardware/GaggiaBoard_V3/KiCad/Project/GaggiaBoard_V3_1.kicad_sch (KiCad schematic)
At the start: 31 parts, among them J1 Display, J14 1x20 Female Header 2.54mm, J15 1x20 Female Header 2.54mm, J2 ToFnLED (Vertical Qwiic), J27 UART1, J4 TC Sensor, J5 2PIN, J6 Pressure TD, J7 Brew & Steam Switches, J8 Scales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

Commit message: KiCad project and model updates
Parts:
- J14, J15: footprint Connector_PinSocket_2.54mm:PinSocket_1x20_P2.54mm_Vertical -> GaggiaBoard_V3:1x20_P2.54mm_Female_Vertical
Changed lines of the file:
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@@
       (effects (font (size 1.27 1.27)) (justify left) hide)
     )
-    (property "Footprint" "Connector_PinSocket_2.54mm:PinSocket_1x20_P2.54mm_Vertical" (at 203.2 53.34 0)
+    (property "Footprint" "GaggiaBoard_V3:1x20_P2.54mm_Female_Vertical" (at 203.2 53.34 0)
       (effects (font (size 1.27 1.27)) hide)
     )
@@
       (effects (font (size 1.27 1.27)) hide)
     )
-    (property "Footprint" "Connector_PinSocket_2.54mm:PinSocket_1x20_P2.54mm_Vertical" (at 172.72 53.34 0)
-      (effects (font (size 1.27 1.27)) hide)
-    )
+    (property "Footprint" "GaggiaBoard_V3:1x20_P2.54mm_Female_Vertical" (at 172.72 53.34 0)
+      (effects (font (size 1.27 1.27)) hide)
+    )
